File: DeckPCB/Deck_Plate_PCB/Deck_Plate_PCB.kicad_pcb (KiCad board)
At the start: 2 copper layers, 124.1 x 104 mm, 65 parts, among them J1 Raspberry_Pi_2_3, J2 NASA_Telemetry_Interface, J3 NASA PWR_Interface, J4 Motor_Inhibit, J5 SunnyBuddy_Inhibit, J6 Batt_JST_Conn, J7 BurWire_Inhibit, P1 Digital, P10 CONN_01X01, P11 CONN_01X01, P12 CONN_01X01, P13 CONN_01X01, P2 Power, P3 Analog, P4 Analog, P5 PWM, P6 PWM, P7 Communication, P8 CONN_01X01, P9 CONN_01X01, Q1 Q_NPN_BCE, Q2 2N7000, Q3 2N7000, U1 Adafruit_INA219_Breakout, U10 LM20, U11 Big_Easy_Driver, U13 LM20, U2 LM2576T-5, U3 D24V25F9, U4 SunnyBuddy_Breakout, U5 LM2576T-5, U6 SF_Logic_Level_Conv, U7 Lidar_RangeFinder, U8 ADXL377

Commit message: Started routing of Deck_Plate_PCB, the main board.
Parts:
- removed C3, C4: 1uF, Capacitor_SMD:C_1206_3216Metric_Pad1.42x1.75mm_HandSolder
- removed D2: 1N5822, Diode_THT:D_DO-201AD_P15.24mm_Horizontal
- removed J4: Motor_Inhibit, Connector_PinHeader_2.54mm:PinHeader_1x02_P2.54mm_Vertical
- removed J5: SunnyBuddy_Inhibit, Connector_PinHeader_2.54mm:PinHeader_1x04_P2.54mm_Vertical
- removed J6: Batt_JST_Conn, Connector_JST:JST_PH_B2B-PH-K_1x02_P2.00mm_Vertical
- removed J7: BurWire_Inhibit, Connector_PinHeader_2.54mm:PinHeader_1x02_P2.54mm_Vertical
- removed Q1: Q_NPN_BCE, Package_TO_SOT_THT:TO-251-3_Vertical
- removed R1: 220, Resistor_THT:R_Axial_DIN0207_L6.3mm_D2.5mm_P10.16mm_Horizontal
- removed R2, R4: 1K, Resistor_THT:R_Axial_DIN0207_L6.3mm_D2.5mm_P10.16mm_Horizontal
- removed R3, R5: 4.7, Resistor_THT:R_Axial_DIN0207_L6.3mm_D2.5mm_P10.16mm_Horizontal
- removed U1: Adafruit_INA219_Breakout, Deck_Plate_PCB:Adafruit_INA219_Breakout_header
- removed U10, U13: LM20, Deck_Plate_PCB:LM20
- removed U11: Big_Easy_Driver, Deck_Plate_PCB:Big_Easy_Driver
- removed U4: SunnyBuddy_Breakout, Deck_Plate_PCB:SunnyBuddy_Breakout
- added J8: Board_to_Board, Connector_PinHeader_2.54mm:PinHeader_1x09_P2.54mm_Vertical, F.Cu at (128.7, 61.3)
- added J9: Power, Connector_PinHeader_2.54mm:PinHeader_1x03_P2.54mm_Vertical, F.Cu at (82.4, 131.9)
- added R6: 10K, Resistor_THT:R_Axial_DIN0207_L6.3mm_D2.5mm_P10.16mm_Horizontal, F.Cu at (91.8, 116.4)
- added R7: 10K, Resistor_THT:R_Axial_DIN0207_L6.3mm_D2.5mm_P10.16mm_Horizontal, F.Cu at (91.9, 121.2)
- added U9: TTL_Camera, Connector_PinHeader_2.54mm:PinHeader_1x04_P2.54mm_Vertical, F.Cu at (82.8, 112.2)
- D1: value LED -> 1N5822; footprint LED_THT:LED_D3.0mm_Clear -> Diode_THT:D_DO-201AD_P12.70mm_Horizontal
- D3: footprint Diode_THT:D_DO-201AD_P15.24mm_Horizontal -> Diode_THT:D_DO-201AD_P12.70mm_Horizontal
- moved D1 212.3 mm to (184.7, 103.2)
- moved H16 50.4 mm to (196.0, 141.0)
- moved J1 50.4 mm to (96.5, 131.8)
- moved R11 50.4 mm to (131.6, 124.9)
- moved H13 50.4 mm to (85.9, 51.0)
- moved H14 50.4 mm to (86.0, 141.0)
- moved H15 50.4 mm to (196.0, 51.0)
- moved J2 50.4 mm to (95.0, 140.4)
- moved P11 50.4 mm to (106.8, 48.9)
- moved P13 50.4 mm to (181.8, 48.9)
- moved P5 50.4 mm to (110.4, 48.9)
- moved P7 50.4 mm to (160.2, 48.9)
- moved C1 50.4 mm to (195.1, 124.1)
- moved C2 50.4 mm to (195.2, 136.4)
- moved C5 50.4 mm to (155.5, 146.5)
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Connections:
- D1 pad 2: GND -> Net-(C1-Pad2)
- J1 pad 10: /TTL_RX -> Net-(J1-Pad10)
- J1 pad 8: /TTL_TX -> Net-(J1-Pad8)
- J2 pad 11: Net-(J2-Pad11) -> /Bit_0
- J2 pad 12: /Bit_2 -> /Bit_1
- J2 pad 13: /Bit_3 -> /Bit_2
- J2 pad 14: /Bit_4 -> /Bit_3
- J2 pad 15: /Bit_5 -> /Bit_4
- J2 pad 16: /Bit_6 -> /Bit_5
- J2 pad 20: /Bit_7 -> /Bit_6
- J2 pad 21: Net-(J2-Pad21) -> /Bit_7
- L1 pad 2: Net-(D2-Pad1) -> Net-(D1-Pad1)
- P2 pad 8: /Vin -> /9V_Bus
- U3 pad 2: /NASA_28V -> /28V_GSE_2
- U5 pad 2: Net-(D2-Pad1) -> Net-(D1-Pad1)
Routing:
- net /5V_Bus_2: track 0.00 -> 302.2 mm, vias 0 -> 2
- net /5V_Bus_1: track 0.00 -> 283.0 mm, vias 0 -> 2
- net /28V_GSE_2: track 0.00 -> 128.2 mm
- net /TTL_RX: track 0.00 -> 117.7 mm
- net /9V_Bus: track 0.00 -> 113.2 mm
- net /TTL_TX: track 0.00 -> 111.4 mm
- net /TE_A: track 0.00 -> 106.1 mm, vias 0 -> 2
- net /TE-RA: track 0.00 -> 99.7 mm
- net /BurnWireSignal: track 0.00 -> 83.3 mm
- net /SolarArrayTemp: track 0.00 -> 68.0 mm
- net /PayloadTemp: track 0.00 -> 64.7 mm
- net /Bit_6: track 0.00 -> 55.7 mm
- net /Step: track 0.00 -> 51.3 mm
- net /TE-RB: track 0.00 -> 48.4 mm
- net Net-(D3-Pad1): track 0.00 -> 47.0 mm, vias 0 -> 1
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