File: DeckPCB/Deck_Plate_PCB/Deck_Plate_PCB.sch (KiCad schematic (older format))
At the start: 19 parts, among them J1 DB37_Female_MountingHoles, J2 DB15_Female_MountingHoles, P1 Digital, P10 CONN_01X01, P11 CONN_01X01, P12 CONN_01X01, P13 CONN_01X01, P2 Power, P3 Analog, P4 Analog, P5 PWM, P6 PWM, P7 Communication, P8 CONN_01X01, P9 CONN_01X01, U1 Adafruit_INA219_Breakout, U2 LM2576T-5, U3 D24V25F9

Commit message: Deleted OnBoardPCB folder, replaced with Deck_Plate_PCB. This should be treated as the MASTER PCB reference from here on out. Added all sensor footprints and symbols as custom parts which are part of a custom DECK_PLATE_PCB library.
Parts:
- removed J1: DB37_Female_MountingHoles, Connector_Dsub:DSUB-37_Female_Vertical_P2.77x2.84mm_MountingHoles, symbol Connector:DB37_Female_MountingHoles
- removed J2: DB15_Female_MountingHoles, Connector_Dsub:DSUB-15_Female_Vertical_P2.77x2.84mm_MountingHoles, symbol Connector:DB15_Female_MountingHoles
- removed U2: LM2576T-5, Package_TO_SOT_THT:TO-220-5_Vertical, symbol Regulator_Switching:LM2576T-5
- added BT?: Battery_Cell, symbol Device:Battery_Cell
- added C? (x2): 1000uF, symbol Device:C
- added C? (x2): 1uF, symbol Device:C
- added D? (x2): 1N5822, Diode_THT:D_DO-201AD_P15.24mm_Horizontal, symbol Diode:1N5822
- added D?: LED, symbol Device:LED
- added J1: Raspberry_Pi_2_3, Connector_PinHeader_2.54mm:PinHeader_2x20_P2.54mm_Vertical, symbol Connector:Raspberry_Pi_2_3
- added J2: DB37_Male_MountingHoles, Connector_Dsub:DSUB-37_Male_Vertical_P2.77x2.84mm_MountingHoles, symbol Connector:DB37_Male_MountingHoles
- added J3: DB15_Male_MountingHoles, Connector_Dsub:DSUB-15_Male_Vertical_P2.77x2.84mm_MountingHoles, symbol Connector:DB15_Male_MountingHoles
- added L? (x2): 100uH, symbol Device:L
- added Q? (x2): 2N7000, Package_TO_SOT_THT:TO-92_Inline, symbol Transistor_FET:2N7000
- added Q?: Q_NPN_BCE, symbol Device:Q_NPN_BCE
- added R?: 220, symbol Device:R
- added R? (x4): 10K, symbol Device:R
- added R? (x4): 5K, symbol Device:R
- added R? (x2): R, symbol Device:R
- added R? (x2): 1K, symbol Device:R
- added U5, U?: LM2576T-5, Package_TO_SOT_THT:TO-220-5_Vertical, symbol Regulator_Switching:LM2576T-5
- added U6: SF_Logic_Level_Conv, Deck_Plate_PCB:SF_Logic_Level_Conv, symbol Deck_Plate_PCB:SF_Logic_Level_Conv
- added U7: LIDAR-LITE_V4_Range, Connector_PinHeader_2.54mm:PinHeader_2x05_P2.54mm_Vertical, symbol Deck_Plate_PCB:LIDAR-LITE_V4_Range
- added U8: ADXL377, Deck_Plate_PCB:ADXL337, symbol Deck_Plate_PCB:ADXL377
- added U?: TTL_Camera, symbol Deck_Plate_PCB:TTL_Camera
- added U? (x2): LM20, symbol Deck_Plate_PCB:LM20
- added U?: Big_Easy_Driver, symbol Deck_Plate_PCB:Big_Easy_Driver
- added U?: Pi_Cam, symbol Deck_Plate_PCB:Pi_Cam
- U4: renamed from U?; footprint (none) -> Deck_Plate_PCB:SunnyBuddy_Breakout
Connections:
- net labels added: 5V_Bus_1, 5V_Bus_2, 9V_Bus, ???, Bit_1, Bit_10, Bit_11, Bit_12, Bit_13, Bit_14, Bit_15, Bit_16, Bit_2, Bit_3, Bit_4, Bit_5, Bit_6, Bit_7, Bit_8, Bit_9, BurnResistorGND, BurnResistorOut, BurnWireSignal, Dir, GPIO_A, GPIO_B, I2C_SCL, I2C_SDA, LED+, Motor_A+, Motor_A-, Motor_B+, Motor_B-, NASA_28V, PayloadTemp, Ribbon_Cable, SolarArrayTemp, Solar_IN+, Solar_IN-, Step, Strobe, TE_A, TE_B, TE_Ra, TE_Rb, TTL_RX, TTL_TX
- wire segments 96 -> 234
- no-connect marks 7 -> 26
Other:
- note added: "- Powering Li-Ion Battery 2200 mAh 3.7V\n- Current and Voltage sensor in-line with Solar input"
- note added: "- TODO: ADD 220uF caps between NASA PWR and GND\n"
- note added: "- TODO: Add TTL Serial Camera Symbol and Footprint\n"
- note added: "- TODO: Define D-Sub connections\n"
- note added: "Burn Wire Circuit\n\n\n\n"
- note added: "NASA Power and Telemetry Interface\n\n"
- note added: "Power Management\n"
- note added: "RaspberryPi Interface\n\n\n"
- note added: "Sensor Management Circuitry\n\n\n"
- note added: "Solar Array Endplate Circuitry\n\n"
- note added: "Solar Charging Circuitry\n\n"
- note added: "Timer Event Handling\n\n\n"
- moved on the sheet: U1, U3, U4

Commit message: Finished all symbol and footprint additions. Added mounting holes for SunnyBuddy, INA219, and ADXL377. Added discrete component footprints. Defined NASA PWR and TELEMETRY pinouts.
Parts:
- added C?: 220uF, Capacitor_SMD:C_1206_3216Metric_Pad1.42x1.75mm_HandSolder, symbol Device:C
- added H? (x4): INA219, MountingHole:MountingHole_2.5mm, symbol Mechanical:MountingHole
- added H? (x4): ADXL377, MountingHole:MountingHole_2.5mm, symbol Mechanical:MountingHole
- added H? (x4): Sunny, MountingHole:MountingHole_2.5mm, symbol Mechanical:MountingHole
- C1, C2, C3, C4: renamed from C?; footprint (none) -> Capacitor_SMD:C_1206_3216Metric_Pad1.42x1.75mm_HandSolder
- D1: renamed from D?; footprint (none) -> LED_THT:LED_D3.0mm_Clear
- J2: value DB37_Male_MountingHoles -> NASA_Telemetry_Interface
- J3: value DB15_Male_MountingHoles -> NASA PWR_Interface
- R1, R10, R11, R12, R13, R2, R3, R4, R5, R6, R7, R8, R9: renamed from R?; footprint (none) -> Resistor_THT:R_Axial_DIN0207_L6.3mm_D2.5mm_P10.16mm_Horizontal
- U10, U13: renamed from U?; footprint (none) -> Deck_Plate_PCB:LM20
- U11: renamed from U?; footprint (none) -> Deck_Plate_PCB:Big_Easy_Driver
- U9: renamed from U?; footprint (none) -> Connector_PinHeader_2.54mm:PinHeader_1x04_P2.54mm_Vertical
- gave numbers to parts that had none: 10
Connections:
- net labels added: 28V_GSE_1, 28V_GSE_2, Analog_1, Analog_10, Analog_2, Analog_3, Analog_4, Analog_5, Analog_6, Analog_7, Analog_8, Analog_9, Bit_16_LSB, Bit_1_MSB, Para_Strobe, RS_DATA, RS_GND, TE-1, TE-2, TE-3, TE-RA, TE-RB
- wire segments 234 -> 237
- no-connect marks 26 -> 30
Other:
- note added: "- TODO: Clarify how the PiCam will be routed concerning the ZIF connection to RaspPi port\n"
- note added: "- TODO: Finish assigning footprints for inductor and other discrete components\n"
- note added: "- TODO: Get with software and confirm signal naming. Go through component by component and make sure output and input names are correct"
- note removed: "- TODO: ADD 220uF caps between NASA PWR and GND\n"
- note removed: "- TODO: Add TTL Serial Camera Symbol and Footprint\n"
- note removed: "- TODO: Define D-Sub connections\n"

Commit message: Updated RaspPi connections based on input from Software. Updated footprints from capacitor and inductor changes. Added inhibit header for batter, motor, and burn-wire.
Parts:
- removed BT1: Battery_Cell, symbol Device:Battery_Cell
- added J4: Inhibit_Header, Connector_PinHeader_2.54mm:PinHeader_1x06_P2.54mm_Vertical, symbol Connector:Conn_01x06_Male
- added U14: Sunny_Batt, Connector_JST:JST_PH_B2B-PH-K_1x02_P2.00mm_Vertical, symbol Deck_Plate_PCB:Sunny_Batt
- C1, C2: footprint Capacitor_SMD:C_1206_3216Metric_Pad1.42x1.75mm_HandSolder -> Deck_Plate_PCB:1000uF_Cap
- C5: renamed from C?; footprint Capacitor_SMD:C_1206_3216Metric_Pad1.42x1.75mm_HandSolder -> Deck_Plate_PCB:220uF_Cap
- L1, L2: footprint (none) -> Inductor_THT:L_Axial_L5.3mm_D2.2mm_P2.54mm_Vertical_Vishay_IM-1
- gave numbers to parts that had none: 12
Connections:
- net labels added: 3v3_Range, Bit_0, Sunny_Batt
- net labels removed: ???, Bit_16
- wire segments 237 -> 228
- no-connect marks 30 -> 43
Other:
- note added: "- TODO get clarification on Burn Wire circuit"
- note added: "- TODO update Burn Wire transistors to new footprint (see PCB Changelog)"
- note removed: "- TODO: Clarify how the PiCam will be routed concerning the ZIF connection to RaspPi port\n"
- moved on the sheet: R3

Commit message: Assigned signals between arduino and sensors based on software input.
Parts:
- removed U14: Sunny_Batt, Connector_JST:JST_PH_B2B-PH-K_1x02_P2.00mm_Vertical, symbol Deck_Plate_PCB:Sunny_Batt
- Q1: footprint (none) -> Package_TO_SOT_THT:TO-251-3_Vertical
- R3, R5: value R -> 4.7
Connections:
- net labels added: Digital_24, Digital_25, Digital_26, Digital_27, Digital_28, Digital_29, Digital_30, Digital_31, Digital_32, Digital_33, Digital_34, Digital_35, Digital_36, Digital_37, Digital_38, Digital_39, Digital_40, Digital_41, Digital_42, Digital_44, Digital_45, Digital_46, Digital_47, Digital_48, Digital_49, TE_RA, TE_RB, Xout, Yout, Zout
- net labels removed: 18(Tx1), 19(Rx1), 22, 23, 24, 25, 26, 27, 28, 29, 30, 31, 32, 33, 34, 35, 36, 37, 38, 39, 40, 41, 42, 43, 44, 45, 46, 47, 48, 49, A10, A14, A15, A8, A9, BurnResistorGND, BurnResistorOut, TE_Ra, TE_Rb
- wire segments 228 -> 231
Other:
- note added: "DONE"
- note added: "Make a 4-pin header (Inhibit_in, GND, Battery_out, GND)\nfor battery charging inhibit"
- note removed: "- TODO get clarification on Burn Wire circuit"
- note removed: "- TODO update Burn Wire transistors to new footprint (see PCB Changelog)"
- moved on the sheet: Q1, R3, R5

Commit message: Updated connections to Logic Level Shifter and LiDAR sensor. Updated inhibit connection scheme.
Parts:
- added J5: SunnyBuddy_Inhibit, Connector_PinHeader_2.54mm:PinHeader_1x04_P2.54mm_Vertical, symbol Connector:Conn_01x04_Male
- added J6: Batt_JST_Conn, Connector_JST:JST_PH_B2B-PH-K_1x02_P2.00mm_Vertical, symbol Connector:Conn_01x02_Male
- added J7: BurWire_Inhibit, Connector_PinHeader_2.54mm:PinHeader_1x02_P2.54mm_Vertical, symbol Connector:Conn_01x02_Male
- J4: value Inhibit_Header -> Motor_Inhibit; footprint Connector_PinHeader_2.54mm:PinHeader_1x06_P2.54mm_Vertical -> Connector_PinHeader_2.54mm:PinHeader_1x02_P2.54mm_Vertical; symbol Connector:Conn_01x06_Male -> Connector:Conn_01x02_Male
Connections:
- net labels added: Batt_In, NASA_Analog_1, NASA_Analog_2, NASA_Analog_3, NASA_Analog_4, Sunny_Batt_Out
- net labels removed: 2(**), 3(**), 3v3_Range, 4(**), Analog_1, Analog_10, Analog_2, Analog_3, Analog_4, Analog_5, Analog_6, Analog_7, Analog_8, Analog_9, Bit_10, Bit_11, Bit_12, Bit_13, Bit_14, Bit_15, Bit_16_LSB, Bit_1_MSB, Bit_8, Bit_9, GPIO_A, GPIO_B, LED+, Sunny_Batt
- wire segments 231 -> 229
- no-connect marks 43 -> 61
Other:
- note added: "Electrical Inhibits\n\n\n\n"
- note removed: "Make a 4-pin header (Inhibit_in, GND, Battery_out, GND)\nfor battery charging inhibit"
- moved on the sheet: C5, J2, J3

Commit message: Initial PCB component placement finished. All mounting holes in place. NOT REPRESENTED: SunnyBuddy, INA219, Electrical inhibits, Motor circuitry, sensor end-panel circuitry. Will create daughter board for these components along with placement for the RaspPi next.
Parts:
- removed H11, H12: ADXL377, MountingHole:MountingHole_2.5mm, symbol Mechanical:MountingHole
- removed H5, H6, H7, H8: INA219, MountingHole:MountingHole_2.5mm, symbol Mechanical:MountingHole
- added H13, H14, H15, H16: Enclos, MountingHole:MountingHole_3.5mm, symbol Mechanical:MountingHole
- H1, H2: value Sunny -> 9V_mount; footprint MountingHole:MountingHole_2.5mm -> MountingHole:MountingHole_2.2mm_M2
- H10, H9: value ADXL377 -> Accel_mount
- H3, H4: value Sunny -> Accel_mount
- J2: footprint Connector_Dsub:DSUB-37_Male_Vertical_P2.77x2.84mm_MountingHoles -> Deck_Plate_PCB:NASA_Telem_37-pin_DSub; symbol Connector:DB37_Male_MountingHoles -> Connector:DB37_Male
- J3: footprint Connector_Dsub:DSUB-15_Male_Vertical_P2.77x2.84mm_MountingHoles -> Deck_Plate_PCB:NASA_PWR_15-pin_DSub; symbol Connector:DB15_Male_MountingHoles -> Connector:DB15_Male
- U7: value LIDAR-LITE_V4_Range -> Lidar_RangeFinder; footprint Connector_PinHeader_2.54mm:PinHeader_2x05_P2.54mm_Vertical -> Connector_PinHeader_2.54mm:PinHeader_1x04_P2.54mm_Vertical
Connections:
- net TE_RA is gone; now on net TE-RA: R8.1
- net TE_RB is gone; now on net TE-RB: R11.1
- net GND: no longer J2.0 (PAD), J3.0 (PAD)
- net Solar_IN+: now also U1.5 (Vin-), U4.2 (Solar_IN+); no longer U1.6 (Vin+), U4.1 (Solar_IN-)
- net Solar_IN-: now also U4.1 (Solar_IN-); no longer U1.5 (Vin-), U4.2 (Solar_IN+)
- net 28V_GSE_1: no longer names the net of J3.1
- net TE-1: no longer names the net of J3.4
- net TE-2: no longer names the net of J3.10 (P10)
- net TE-3: no longer names the net of J3.11 (P111)
- new net SolarCell+: U1.6 (Vin+)
- no-connect marks 61 -> 59
Other:
- moved on the sheet: H1, H10, H2, H3, H4, H9
Changed lines of the file:
@@
 U 1 1 5E458126
 P 450 5350
-F 0 "U7" H 1850 5550 50  0000 C CNN
-F 1 "LIDAR-LITE_V4_Range" H 1550 6450 50  0000 C CNN
-F 2 "Connector_PinHeader_2.54mm:PinHeader_2x05_P2.54mm_Vertical" H 1900 6300 50  0001 C CNN
+F 0 "U7" H 1850 6050 50  0000 C CNN
+F 1 "Lidar_RangeFinder" H 1550 6450 50  0000 C CNN
+F 2 "Connector_PinHeader_2.54mm:PinHeader_1x04_P2.54mm_Vertical" H 1900 6300 50  0001 C CNN
 F 3 "https://static.garmin.com/pumac/LIDAR-Lite%20LED%20v4%20Instructions_EN-US.pdf" H 1900 6300 50  0001 C CNN
 	1    450  5350
@@
 $EndComp
 $Comp
-L Connector:DB37_Male_MountingHoles J2
+L Connector:DB37_Male J2
 U 1 1 5E4749AA
 P 2600 7400
 F 0 "J2" V 2825 7368 50  0000 C CNN
 F 1 "NASA_Telemetry_Interface" V 2916 7368 50  0000 C CNN
-F 2 "Connector_Dsub:DSUB-37_Male_Vertical_P2.77x2.84mm_MountingHoles" H 2600 7400 50  0001 C CNN
+F 2 "Deck_Plate_PCB:NASA_Telem_37-pin_DSub" H 2600 7400 50  0001 C CNN
 F 3 " ~" H 2600 7400 50  0001 C CNN
 	1    2600 7400
@@
 $EndComp
 $Comp
-L Connector:DB15_Male_MountingHoles J3
+L Connector:DB15_Male J3
 U 1 1 5E47F177
 P 5950 7400
 F 0 "J3" V 6149 7355 50  0000 C CNN
 F 1 "NASA PWR_Interface" V 6240 7355 50  0000 C CNN
-F 2 "Connector_Dsub:DSUB-15_Male_Vertical_P2.77x2.84mm_MountingHoles" H 5950 7400 50  0001 C CNN
+F 2 "Deck_Plate_PCB:NASA_PWR_15-pin_DSub" H 5950 7400 50  0001 C CNN
 F 3 " ~" H 5950 7400 50  0001 C CNN
 	1    5950 7400
@@
 	1100 3100 1000 3100
 Text Label 1000 3000 2    50   ~ 0
+Solar_IN-
+Text Label 1000 3100 2    50   ~ 0
 Solar_IN+
-Text Label 1000 3100 2    50   ~ 0
-Solar_IN-
 $Comp
 L power:GND #PWR0104
@@
 Wire Wire Line
 	2500 3500 2600 3500
-Text Label 2600 3000 0    50   ~ 0
-Solar_IN+
-Text Label 2600 3100 0    50   ~ 0
-Solar_IN-
 Text Label 2600 3550 0    50   ~ 0
 5V_Bus_1
@@
 Text Label 2950 4900 2    50   ~ 0
 I2C_SDA
-NoConn ~ 1050 5000
-NoConn ~ 1050 4850
-NoConn ~ 2000 4850
-NoConn ~ 2000 5000
 $Comp
 L power:GND #PWR0108
@@
 5V_Bus_2
 Text Label 7500 3900 0    50   ~ 0
-TE_RB
+TE-RB
 Wire Wire Line
 	7850 4650 8100 4650
@@
 5V_Bus_2
 Text Label 6450 3900 0    50   ~ 0
-TE_RA
+TE-RA
 Wire Wire Line
 	6800 4650 7050 4650
@@
 Wire Notes Line
 	5550 5200 5550 6550
-Text Label 5250 7100 1    50   ~ 0
-28V_GSE_1
 Text Label 5450 7100 1    50   ~ 0
 TE-RA
 Text Label 5650 7100 1    50   ~ 0
 TE-RB
-Text Label 5850 7100 1    50   ~ 0
-TE-1
 $Comp
 L power:GND #PWR0131
@@
 Text Label 5350 7100 1    50   ~ 0
 28V_GSE_2
-Text Label 5550 7100 1    50   ~ 0
-TE-2
-Text Label 5750 7100 1    50   ~ 0
-TE-3
 $Comp
 L power:GND #PWR0135
@@
 	4800 6650 5350 6650
 $Comp
-L power:GND #PWR0144
-U 1 1 5E62467C
-P 5050 7400
-F 0 "#PWR0144" H 5050 7150 50  0001 C CNN
-F 1 "GND" V 5055 7272 50  0000 R CNN
-F 2 "" H 5050 7400 50  0001 C CNN
-F 3 "" H 5050 7400 50  0001 C CNN
-	1    5050 7400
-	1    0    0    -1
-$EndComp
-$Comp
-L power:GND #PWR0145
-U 1 1 5E624BAC
-P 600 7400
-F 0 "#PWR0145" H 600 7150 50  0001 C CNN
-F 1 "GND" V 605 7272 50  0000 R CNN
-F 2 "" H 600 7400 50  0001 C CNN
-F 3 "" H 600 7400 50  0001 C CNN
-	1    600  7400
-	1    0    0    -1
-$EndComp
-$Comp
-L Mechanical:MountingHole H5
-U 1 1 5E63B3F7
-P 9350 6150
-F 0 "H5" H 9250 6104 50  0000 R CNN
-F 1 "INA219" H 9250 6195 50  0000 R CNN
-F 2 "MountingHole:MountingHole_2.5mm" H 9350 6150 50  0001 C CNN
-F 3 "~" H 9350 6150 50  0001 C CNN
-	1    9350 6150
-	-1   0    0    1
-$EndComp
-$Comp
-L Mechanical:MountingHole H6
-U 1 1 5E63DA2B
-P 9350 6350
-F 0 "H6" H 9250 6304 50  0000 R CNN
-F 1 "INA219" H 9250 6395 50  0000 R CNN
-F 2 "MountingHole:MountingHole_2.5mm" H 9350 6350 50  0001 C CNN
-F 3 "~" H 9350 6350 50  0001 C CNN
-	1    9350 6350
-	-1   0    0    1
-$EndComp
-$Comp
-L Mechanical:MountingHole H7
-U 1 1 5E63DE75
-P 9800 6150
-F 0 "H7" H 9700 6104 50  0000 R CNN
-F 1 "INA219" H 9700 6195 50  0000 R CNN
-F 2 "MountingHole:MountingHole_2.5mm" H 9800 6150 50  0001 C CNN
-F 3 "~" H 9800 6150 50  0001 C CNN
-	1    9800 6150
-	-1   0    0    1
-$EndComp
-$Comp
-L Mechanical:MountingHole H8
-U 1 1 5E63E369
-P 9800 6350
-F 0 "H8" H 9700 6304 50  0000 R CNN
-F 1 "INA219" H 9700 6395 50  0000 R CNN
-F 2 "MountingHole:MountingHole_2.5mm" H 9800 6350 50  0001 C CNN
-F 3 "~" H 9800 6350 50  0001 C CNN
-	1    9800 6350
-	-1   0    0    1
-$EndComp
-$Comp
 L Mechanical:MountingHole H9
 U 1 1 5E63E671
-P 10250 6150
-F 0 "H9" H 10150 6104 50  0000 R CNN
-F 1 "ADXL377" H 10150 6195 50  0000 R CNN
-F 2 "MountingHole:MountingHole_2.5mm" H 10250 6150 50  0001 C CNN
-F 3 "~" H 10250 6150 50  0001 C CNN
-	1    10250 6150
+P 10600 6150
+F 0 "H9" H 10500 6104 50  0000 R CNN
+F 1 "Accel_mount" H 10500 6195 50  0000 R CNN
+F 2 "MountingHole:MountingHole_2.5mm" H 10600 6150 50  0001 C CNN
+F 3 "~" H 10600 6150 50  0001 C CNN
+	1    10600 6150
 	-1   0    0    1
 $EndComp
@@
 L Mechanical:MountingHole H10
 U 1 1 5E63EB24
-P 10250 6350
-F 0 "H10" H 10150 6304 50  0000 R CNN
-F 1 "ADXL377" H 10150 6395 50  0000 R CNN
-F 2 "MountingHole:MountingHole_2.5mm" H 10250 6350 50  0001 C CNN
-F 3 "~" H 10250 6350 50  0001 C CNN
-	1    10250 6350
-	-1   0    0    1
-$EndComp
-$Comp
-L Mechanical:MountingHole H11
-U 1 1 5E63EEC6
-P 10750 6150
-F 0 "H11" H 10650 6104 50  0000 R CNN
-F 1 "ADXL377" H 10650 6195 50  0000 R CNN
-F 2 "MountingHole:MountingHole_2.5mm" H 10750 6150 50  0001 C CNN
-F 3 "~" H 10750 6150 50  0001 C CNN
-	1    10750 6150
-	-1   0    0    1
-$EndComp
-$Comp
-L Mechanical:MountingHole H12
-U 1 1 5E63F40C
-P 10750 6350
-F 0 "H12" H 10650 6304 50  0000 R CNN
-F 1 "ADXL377" H 10650 6395 50  0000 R CNN
-F 2 "MountingHole:MountingHole_2.5mm" H 10750 6350 50  0001 C CNN
-F 3 "~" H 10750 6350 50  0001 C CNN
-	1    10750 6350
+P 10600 6350
+F 0 "H10" H 10500 6304 50  0000 R CNN
+F 1 "Accel_mount" H 10500 6395 50  0000 R CNN
+F 2 "MountingHole:MountingHole_2.5mm" H 10600 6350 50  0001 C CNN
+F 3 "~" H 10600 6350 50  0001 C CNN
+	1    10600 6350
 	-1   0    0    1
 $EndComp
@@
 L Mechanical:MountingHole H3
 U 1 1 5E63F891
-P 8950 6150
-F 0 "H3" H 8850 6104 50  0000 R CNN
-F 1 "Sunny" H 8850 6195 50  0000 R CNN
-F 2 "MountingHole:MountingHole_2.5mm" H 8950 6150 50  0001 C CNN
-F 3 "~" H 8950 6150 50  0001 C CNN
-	1    8950 6150
+P 9900 6150
+F 0 "H3" H 9800 6104 50  0000 R CNN
+F 1 "Accel_mount" H 9800 6195 50  0000 R CNN
+F 2 "MountingHole:MountingHole_2.5mm" H 9900 6150 50  0001 C CNN
+F 3 "~" H 9900 6150 50  0001 C CNN
+	1    9900 6150
 	-1   0    0    1
 $EndComp
@@
 L Mechanical:MountingHole H4
 U 1 1 5E63FD37
-P 8950 6350
-F 0 "H4" H 8850 6304 50  0000 R CNN
-F 1 "Sunny" H 8850 6395 50  0000 R CNN
-F 2 "MountingHole:MountingHole_2.5mm" H 8950 6350 50  0001 C CNN
-F 3 "~" H 8950 6350 50  0001 C CNN
-	1    8950 6350
+P 9900 6350
+F 0 "H4" H 9800 6304 50  0000 R CNN
+F 1 "Accel_mount" H 9800 6395 50  0000 R CNN
+F 2 "MountingHole:MountingHole_2.5mm" H 9900 6350 50  0001 C CNN
+F 3 "~" H 9900 6350 50  0001 C CNN
+	1    9900 6350
 	-1   0    0    1
 $EndComp
@@
 L Mechanical:MountingHole H2
 U 1 1 5E6401D5
-P 8550 6350
-F 0 "H2" H 8450 6304 50  0000 R CNN
-F 1 "Sunny" H 8450 6395 50  0000 R CNN
-F 2 "MountingHole:MountingHole_2.5mm" H 8550 6350 50  0001 C CNN
-F 3 "~" H 8550 6350 50  0001 C CNN
-	1    8550 6350
+P 9300 6350
+F 0 "H2" H 9200 6304 50  0000 R CNN
+F 1 "9V_mount" H 9200 6395 50  0000 R CNN
+F 2 "MountingHole:MountingHole_2.2mm_M2" H 9300 6350 50  0001 C CNN
+F 3 "~" H 9300 6350 50  0001 C CNN
+	1    9300 6350
 	-1   0    0    1
 $EndComp
@@
 L Mechanical:MountingHole H1
 U 1 1 5E640799
-P 8550 6150
-F 0 "H1" H 8450 6104 50  0000 R CNN
-F 1 "Sunny" H 8450 6195 50  0000 R CNN
-F 2 "MountingHole:MountingHole_2.5mm" H 8550 6150 50  0001 C CNN
-F 3 "~" H 8550 6150 50  0001 C CNN
-	1    8550 6150
+P 9300 6150
+F 0 "H1" H 9200 6104 50  0000 R CNN
+F 1 "9V_mount" H 9200 6195 50  0000 R CNN
+F 2 "MountingHole:MountingHole_2.2mm_M2" H 9300 6150 50  0001 C CNN
+F 3 "~" H 9300 6150 50  0001 C CNN
+	1    9300 6150
 	-1   0    0    1
 $EndComp
@@
 Text Label 2150 4400 0    50   ~ 0
 5V_Bus_1
-NoConn ~ 2000 4700
-NoConn ~ 1050 4700
 Text Notes 3350 4150 0    50   ~ 0
 DONE
-Text Notes 700  4800 0    50   ~ 0
+Text Notes 1300 4750 0    50   ~ 0
 DONE
 Text Notes 6900 5400 0    50   ~ 0
@@
 NoConn ~ 2700 7100
 NoConn ~ 2800 7100
+Text Notes 4450 6250 0    50   ~ 0
+DONE
+NoConn ~ 5250 7100
+NoConn ~ 5850 7100
+NoConn ~ 5750 7100
+NoConn ~ 5550 7100
+Text Notes 1500 3600 0    50   ~ 0
+DONE
+$Comp
+L Mechanical:MountingHole H15
+U 1 1 5E5EBE19
+P 8850 6350
+F 0 "H15" H 8750 6304 50  0000 R CNN
+F 1 "Enclos" H 8750 6395 50  0000 R CNN
+F 2 "MountingHole:MountingHole_3.5mm" H 8850 6350 50  0001 C CNN
+F 3 "~" H 8850 6350 50  0001 C CNN
+	1    8850 6350
+	-1   0    0    1
+$EndComp
+$Comp
+L Mechanical:MountingHole H16
+U 1 1 5E5EC212
+P 8850 6150
+F 0 "H16" H 8750 6104 50  0000 R CNN
+F 1 "Enclos" H 8750 6195 50  0000 R CNN
+F 2 "MountingHole:MountingHole_3.5mm" H 8850 6150 50  0001 C CNN
+F 3 "~" H 8850 6150 50  0001 C CNN
+	1    8850 6150
+	-1   0    0    1
+$EndComp
+$Comp
+L Mechanical:MountingHole H14
+U 1 1 5E5EC76A
+P 8400 6350
+F 0 "H14" H 8300 6304 50  0000 R CNN
+F 1 "Enclos" H 8300 6395 50  0000 R CNN
+F 2 "MountingHole:MountingHole_3.5mm" H 8400 6350 50  0001 C CNN
+F 3 "~" H 8400 6350 50  0001 C CNN
+	1    8400 6350
+	-1   0    0    1
+$EndComp
+$Comp
+L Mechanical:MountingHole H13
+U 1 1 5E5ECA7F
+P 8400 6150
+F 0 "H13" H 8300 6104 50  0000 R CNN
+F 1 "Enclos" H 8300 6195 50  0000 R CNN
+F 2 "MountingHole:MountingHole_3.5mm" H 8400 6150 50  0001 C CNN
+F 3 "~" H 8400 6150 50  0001 C CNN
+	1    8400 6150
+	-1   0    0    1
+$EndComp
+Text Label 2600 3000 0    50   ~ 0
+SolarCell+
+Text Label 2600 3100 0    50   ~ 0
+Solar_IN+
 $EndSCHEMATC
